Commit message: add YOLOv8

File: description/camera.xacro (robot description, xacro)
@@ -34,4 +34,20 @@
     <child link="camera_frame"/>
   </joint>
+  <!-- Camera Field of View Boundary Box -->
+  <link name="camera_view_boundary">
+    <visual>
+      <origin xyz="0.6 0 0" rpy="0 0 0"/>  <!-- 60cm forward -->
+      <geometry>
+        <box size="0.01 0.85 0.65"/>  <!-- Thin box, width x height based on FOV -->
+      </geometry>
+      <material name="camera_boundary">
+        <color rgba="1.0 0.8 0.0 0.4"/>  <!-- Orange-yellow, 40% transparent -->
+      </material>
+    </visual>
+  </link>
+  <joint name="camera_view_boundary_joint" type="fixed">
+    <parent link="camera_link"/>
+    <child link="camera_view_boundary"/>
+  </joint>
   <gazebo reference="camera_link">
     <material>Gazebo/Green</material>
